File: linht-hw.kicad_pcb (KiCad board)
At the start: 4 copper layers, 45.5 x 96 mm, 176 parts, among them IC1 SX1255IWLTRT, J1 Antenna, J10 GND, J11 Keyboard, J12 USB_C, J13 2.5mm, J14 3.5mm, J15 SPEAKER, J2 Battery connector, J3 GND spring, J4 SPEAKER, J5 LCD, J6 GND, J7 GND, J8 PTT, J9 BTN_2, Q1 BSS138, Q2 BSS138, Q3 BSS138, Q4 BSS138, Q5 BSS138, SW2 10k, U1 MCM-iMX93, U2 BGS12P2L6, U3 TPS562203, U4 TPS562203, U5 74AHC1G86, U6 WM8960, U7 MAX9814, U8 USBLC6-2SC6, Y1 32MHz, Y2 12.288M

Commit message: Attempt to add GNSS Quectel LG77L module
Adding rst/wkp lines + board cleanup

removed lvl shifter and LDO - added passive elements gnss rf-in
Parts:
- added C68: , Capacitor_SMD:C_0402_1005Metric, F.Cu at (142.3, 125.0)
- added C69: , Capacitor_SMD:C_0402_1005Metric, F.Cu at (142.3, 126.0)
- added J4: U.FL_Molex_MCRF_73412-0110_Vertical, Connector_Coaxial:U.FL_Molex_MCRF_73412-0110_Vertical, F.Cu at (143.1, 121.3)
- added R63: , Resistor_SMD:R_0402_1005Metric, F.Cu at (143.8, 125.5)
- added U12: XCVR_LG77L, Quectel LG77:XCVR_LG77L, B.Cu at (140.2, 130.3)
- added Y3: Crystal_SMD_3215-2Pin_3.2x1.5mm, Crystal:Crystal_SMD_3215-2Pin_3.2x1.5mm, B.Cu at (143.0, 136.4)
- moved Q5 2.56 mm to (143.6, 135.1)
- moved R44 2.56 mm to (143.5, 132.0)
- moved R45 2.56 mm to (142.5, 132.0)
- moved R43 0.95 mm to (141.0, 137.9)
Connections:
- U1 pad 130: unconnected-(U1-Pad130) -> GNSS/UART2_RX
- U1 pad 133: unconnected-(U1-Pad133) -> GNSS/UART2_TX
- U1 pad 69: unconnected-(U1-GPIO3_IO[2]-Pad69) -> /GNSS/RST_GNSS
- U1 pad 70: unconnected-(U1-GPIO3_IO[1]-Pad70) -> /GNSS/WAKEUP_GNSS
- U1 pad 84: unconnected-(U1-Pad84) -> GNSS/UART3_TX
- U1 pad 88: unconnected-(U1-Pad88) -> GNSS/UART3_RX
Routing:
- net +3V3: track 48.6 -> 85.7 mm, vias 28 -> 29
- net VDD: track 42.9 -> 67.9 mm, vias 4 -> 9
- net /GNSS/RST_GNSS: track 0.00 -> 22.2 mm, vias 0 -> 1
- net /GNSS/WAKEUP_GNSS: track 0.00 -> 20.4 mm, vias 0 -> 1
- net (no net): track 0.00 -> 10.00 mm
- net /GNSS/RF_IN: track 0.00 -> 7.59 mm, vias 0 -> 1
- net GNSS/UART3_TX: track 0.00 -> 4.54 mm, vias 0 -> 1
- net GNSS/UART3_RX: track 0.00 -> 3.64 mm, vias 0 -> 1
- net Net-(J11-Pin_2): track 25.3 -> 27.3 mm
- net Net-(Q5-D): track 1.47 -> 3.12 mm
- net /Keyboard/SIDE_BTN: track 76.6 -> 77.4 mm
- net /Audio/I2C_SCL: track 20.4 -> 19.7 mm
- net /Audio/I2C_SDA: track 20.6 -> 19.9 mm
- net /Audio/I2S_WS_IN: track 57.7 -> 57.1 mm
- net GND: vias 239 -> 234
