File: linht-hw.kicad_sch (KiCad schematic)
At the start: 0 parts

Commit message: Attempt to add GNSS Quectel LG77L module
Adding rst/wkp lines + board cleanup

removed lvl shifter and LDO - added passive elements gnss rf-in
Other:
- added sheet GNSS (gnss.kicad_sch)
Changed lines of the file:
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@@
+		)
+	)
+	(hierarchical_label "UART3_TX"
+		(shape output)
+		(at 163.83 30.48 180)
+		(effects
+			(font
+				(size 1.27 1.27)
+			)
+			(justify right)
+		)
+	)
+	(hierarchical_label "UART3_RX"
+		(shape input)
+		(at 163.83 33.02 180)
+		(effects
+			(font
+				(size 1.27 1.27)
+			)
+			(justify right)
 		)
 	)
@@
 	)
 	(sheet
-		(at 127 38.1)
-		(size 36.83 91.44)
+		(at 127 26.67)
+		(size 36.83 102.87)
 		(exclude_from_sim no)
 		(in_bom yes)
@@
 		)
 		(property "Sheetname" "SoC"
-			(at 127 37.3884 0)
+			(at 127 25.9584 0)
 			(effects
 				(font
@@
 				)
 			)
+		)
+	)
+	(sheet
+		(at 209.55 26.67)
+		(size 25.4 20.32)
+		(exclude_from_sim no)
+		(in_bom yes)
+		(on_board yes)
+		(dnp no)
+		(fields_autoplaced yes)
+		(stroke
+			(width 0.1524)
+			(type solid)
+		)
+		(fill
+			(color 255 255 194 1.0000)
+		)
+		(property "Sheetname" "GNSS"
+			(at 209.55 25.9584 0)
+			(effects
+				(font
+					(size 1.27 1.27)
+				)
+				(justify left bottom)
+			)
+		)
+		(property "Sheetfile" "gnss.kicad_sch"
+			(at 209.55 47.5746 0)
+			(effects
+				(font
+					(size 1.27 1.27)
+				)
+				(justify left top)
+			)
+		)
+		(instances
+			(project "linht-hw"
+				(path "/73efc1fc-21f6-4aef-9f73-508fe18fa32e"
+					(page "9")
+				)
+			)
