File: soc.kicad_sch (KiCad schematic)
At the start: 7 parts, among them U1 MCM-iMX93

Commit message: Attempt to add GNSS Quectel LG77L module
Adding rst/wkp lines + board cleanup

removed lvl shifter and LDO - added passive elements gnss rf-in
Parts:
- renumbered U1 to GPIO4_IO[5]1
Connections:
- net WAKEUP_GNSS: now reaches GPIO4_IO[5]1.69 (GPIO3_IO[2])
- net RST_GNSS: now reaches GPIO4_IO[5]1.70 (GPIO3_IO[1])
- net UART3_TX: now reaches GPIO4_IO[5]1.84 (UART3_TX)
- net UART3_RX: now reaches GPIO4_IO[5]1.88 (UART3_RX)
- no-connect marks 83 -> 81
Changed lines of the file:
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@@
-	)
-	(no_connect
-		(at 134.62 171.45)
 	)
 	(no_connect
@@
 	(no_connect
 		(at 44.45 133.35)
-	)
-	(no_connect
-		(at 137.16 171.45)
 	)
 	(bus_entry
@@
 	(wire
 		(pts
+			(xy 137.16 171.45) (xy 137.16 177.8)
+		)
+		(stroke
+			(width 0)
+			(type default)
+		)
+	)
+	(wire
+		(pts
 			(xy 88.9 40.64) (xy 88.9 45.72)
 		)
@@
 	(wire
 		(pts
+			(xy 143.51 105.41) (xy 148.59 105.41)
+		)
+		(stroke
+			(width 0)
+			(type default)
+		)
+	)
+	(wire
+		(pts
 			(xy 143.51 74.93) (xy 148.59 74.93)
 		)
@@
 	(wire
 		(pts
+			(xy 143.51 115.57) (xy 148.59 115.57)
+		)
+		(stroke
+			(width 0)
+			(type default)
+		)
+	)
+	(wire
+		(pts
 			(xy 209.55 68.58) (xy 209.55 69.85)
 		)
@@
 		(pts
 			(xy 91.44 171.45) (xy 91.44 175.26)
+		)
+		(stroke
+			(width 0)
+			(type default)
+		)
+	)
+	(wire
+		(pts
+			(xy 134.62 171.45) (xy 134.62 177.8)
 		)
 		(stroke
@@
 		)
 	)
+	(hierarchical_label "UART3_RX"
+		(shape input)
+		(at 148.59 105.41 0)
+		(effects
+			(font
+				(size 1.27 1.27)
+			)
+			(justify left)
+		)
+	)
 	(hierarchical_label "SPI_CS_RF"
 		(shape output)
@@
 		)
 	)
+	(hierarchical_label "UART3_TX"
+		(shape output)
+		(at 148.59 115.57 0)
+		(effects
+			(font
+				(size 1.27 1.27)
+			)
+			(justify left)
+		)
+	)
 	(hierarchical_label "I2S1_WS"
 		(shape output)
@@
 		)
 	)
+	(hierarchical_label "WAKEUP_GNSS"
+		(shape output)
+		(at 134.62 177.8 270)
+		(effects
+			(font
+				(size 1.27 1.27)
+			)
+			(justify right)
+		)
+	)
 	(hierarchical_label "LED_B"
 		(shape output)
@@
 			)
 			(justify left)
+		)
+	)
+	(hierarchical_label "RST_GNSS"
+		(shape output)
+		(at 137.16 177.8 270)
+		(effects
+			(font
+				(size 1.27 1.27)
+			)
+			(justify right)
 		)
 	)
@@
 		(on_board yes)
 		(dnp no)
-		(property "Reference" "U1"
+		(property "Reference" "GPIO4_IO[5]1"
 			(at 93.98 104.2557 0)
 			(effects
@@
 			(project ""
 				(path "/73efc1fc-21f6-4aef-9f73-508fe18fa32e/9e50fe40-00b4-48a0-8ec6-ce79209e6a2d"
-					(reference "U1")
+					(reference "GPIO4_IO[5]1")
 					(unit 1)
 				)
